File: Hardware/SparkFun_SSOP16_Breakout.sch (EAGLE design)
At the start: 11 parts, among them U1 SSOP16, U2 SSOP16

Commit message: Checklist updates.
Package outline to 8 mil.
Version to V21.
Other:
- note added: "V21"
- note removed: "V20"
Changed lines of the file:
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@@
 <sheet>
 <plain>
-<text x="238.76" y="7.62" size="2.54" layer="94" font="vector">V20</text>
+<text x="238.76" y="7.62" size="2.54" layer="94" font="vector">V21</text>
 <text x="165.1" y="7.62" size="2.54" layer="94" font="vector">Byron Jacquot</text>
 </plain>
